Commit message: added go1_description related file, copied from a1 config for go1

File: legged_examples/legged_unitree/legged_unitree_description/urdf/go1/const.xacro (robot description, xacro)
@@ -19,4 +19,8 @@
     <xacro:property name="stick_radius" value="0.01"/>
     <xacro:property name="stick_length" value="0.2"/>
+    <!-- copied missing property from a1-->
+    <xacro:property name="thigh_shoulder_y_offset" value="-0.008"/>
+    <xacro:property name="thigh_x_offset" value="-0.015"/>
+    <xacro:property name="calf_x_offset" value="0.0"/>
     <!-- kinematic value -->
     <xacro:property name="thigh_offset" value="0.08"/>
@@ -26,5 +30,5 @@
     <xacro:property name="leg_offset_x" value="0.1881"/>
     <xacro:property name="leg_offset_y" value="0.04675"/>
-    <!-- <xacro:property name="trunk_offset_z" value="0.01675"/> -->
+    <xacro:property name="trunk_offset_z" value="0.01675"/>
     <xacro:property name="hip_offset" value="0.08"/>
     <!-- offset of link and rotor locations (left front) -->
@@ -50,14 +54,14 @@
     <xacro:property name="damping" value="0.01"/>
     <xacro:property name="friction" value="0.2"/>
-    <xacro:property name="hip_position_max" value="0.863"/>
-    <xacro:property name="hip_position_min" value="-0.863"/>
+    <xacro:property name="hip_max" value="0.863"/>
+    <xacro:property name="hip_min" value="-0.863"/>
     <xacro:property name="hip_velocity_max" value="30.1"/>
     <xacro:property name="hip_torque_max" value="23.7"/>
-    <xacro:property name="thigh_position_max" value="4.501"/>
-    <xacro:property name="thigh_position_min" value="-0.686"/>
+    <xacro:property name="thigh_max" value="4.501"/>
+    <xacro:property name="thigh_min" value="-0.686"/>
     <xacro:property name="thigh_velocity_max" value="30.1"/>
     <xacro:property name="thigh_torque_max" value="23.7"/>
-    <xacro:property name="calf_position_max" value="-0.888"/>
-    <xacro:property name="calf_position_min" value="-2.818"/>
+    <xacro:property name="calf_max" value="-0.888"/>
+    <xacro:property name="calf_min" value="-2.818"/>
     <xacro:property name="calf_velocity_max" value="20.06"/>
     <xacro:property name="calf_torque_max" value="35.55"/>
