Commit message: add d435 to go1

File: legged_examples/legged_unitree/legged_unitree_description/urdf/robot.xacro (robot description, xacro)
@@ -7,4 +7,8 @@
     <xacro:include filename="$(find legged_unitree_description)/urdf/common/imu.xacro"/>
     <xacro:include filename="$(find legged_unitree_description)/urdf/$(arg robot_type)/const.xacro"/>
+    <xacro:include filename="$(find realsense2_description)/urdf/_d435.urdf.xacro" />
+        <xacro:sensor_d435 name="camera" parent="base">
+        <origin xyz="0.25 0 0.1" rpy="0 0 0"/>
+    </xacro:sensor_d435>
     <link name="base">
         <visual>
